File: TelescopeController/12v_switching.kicad_sch (KiCad schematic)
At the start: 10 parts, among them Q1 DMN63D8LW-13, Q2 AO3423

Commit message: add telescope controller v2
Parts:
- removed D3: SML-LX0805GC-TR, LED_SMD:LED_0805_2012Metric_Pad1.15x1.40mm_HandSolder, symbol Device:LED
- removed Q2: AO3423, AO3423:SOT95P280X125-3N, symbol AO3423:AO3423
- added D13: LED, LED_THT:LED_D3.0mm, symbol Device:LED
- added Q2: DMP3099L-7, DMP3099L-7:SOT96P240X115-3N, symbol DMP3099L-7:DMP3099L-7
- F2: value 1A -> 1.5A
- R2: value 100R -> 1k
- R20: value 490R -> 1k
Connections:
- net GND: now also D13.1 (K)
- net OUT: now also Q2.3 (D)
- net at Q1.3, R2.2, TP1.1: now also Q2.1 (G)
- net at R20.2: now also D13.2 (A)
- net at F2.2, R2.1: now also Q2.2 (S)
Other:
- note added: "https://tinyurl.com/2d8vguqs"
Changed lines of the file:
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@@
+    (stroke (width 0) (type default))
+  )
+  (wire (pts (xy 114.3 83.82) (xy 116.84 83.82))
+    (stroke (width 0) (type default))
+  )
+  (wire (pts (xy 137.16 54.61) (xy 137.16 66.04))
+    (stroke (width 0) (type default))
+  )
+  (wire (pts (xy 153.67 60.96) (xy 153.67 66.04))
+    (stroke (width 0) (type default))
+  )
+  (wire (pts (xy 137.16 66.04) (xy 153.67 66.04))
+    (stroke (width 0) (type default))
+  )
+  (wire (pts (xy 161.29 39.37) (xy 161.29 55.88))
+    (stroke (width 0) (type default))
+  )
+  (wire (pts (xy 121.92 97.79) (xy 121.92 102.87))
     (stroke (width 0) (type default))
   )
@@
     (stroke (width 0) (type default))
   )
-  (wire (pts (xy 114.3 83.82) (xy 116.84 83.82))
-    (stroke (width 0) (type default))
-  )
-  (wire (pts (xy 137.16 54.61) (xy 137.16 66.04))
-    (stroke (width 0) (type default))
-  )
-  (wire (pts (xy 137.16 66.04) (xy 153.67 66.04))
-    (stroke (width 0) (type default))
-  )
-  (wire (pts (xy 161.29 39.37) (xy 161.29 55.88))
-    (stroke (width 0) (type default))
-  )
-  (wire (pts (xy 121.92 97.79) (xy 121.92 102.87))
-    (stroke (width 0) (type default))
-  )
   (wire (pts (xy 137.16 46.99) (xy 137.16 39.37))
     (stroke (width 0) (type default))
@@
   (wire (pts (xy 116.84 83.82) (xy 121.92 83.82))
     (stroke (width 0) (type default))
+  )
+  (text "https://tinyurl.com/2d8vguqs" (at 92.71 58.928 0)
+    (effects (font (size 1.27 1.27)) (justify left bottom))
   )
   (hierarchical_label "IN" (shape input) (at 114.3 83.82 180) (fields_autoplaced)
@@
       (effects (font (size 1.27 1.27)) (justify left))
     )
-    (property "Value" "490R" (at 163.83 92.71 0)
+    (property "Value" "1k" (at 163.83 92.71 0)
       (effects (font (size 1.27 1.27)) (justify left))
     )
@@
     )
   )
+  (symbol (lib_id "DMP3099L-7:DMP3099L-7") (at 153.67 60.96 0) (mirror x) (unit 1)
+    (in_bom yes) (on_board yes) (dnp no)
+    (property "Reference" "Q2" (at 165.608 64.77 0)
+      (effects (font (size 1.27 1.27)) (justify left))
+    )
+    (property "Value" "DMP3099L-7" (at 165.608 62.23 0)
+      (effects (font (size 1.27 1.27)) (justify left))
+    )
+    (property "Footprint" "DMP3099L-7:SOT96P240X115-3N" (at 165.1 -37.77 0)
+      (effects (font (size 1.27 1.27)) (justify left top) hide)
+    )
+    (property "Datasheet" "https://www.diodes.com//assets/Datasheets/DMP3099L.pdf" (at 165.1 -137.77 0)
+      (effects (font (size 1.27 1.27)) (justify left top) hide)
+    )
+    (property "Height" "1.15" (at 165.1 -337.77 0)
+      (effects (font (size 1.27 1.27)) (justify left top) hide)
+    )
+    (property "Manufacturer_Name" "Diodes Incorporated" (at 165.1 -437.77 0)
+      (effects (font (size 1.27 1.27)) (justify left top) hide)
+    )
+    (property "Manufacturer_Part_Number" "DMP3099L-7" (at 165.1 -537.77 0)
+      (effects (font (size 1.27 1.27)) (justify left top) hide)
+    )
+    (property "Mouser Part Number" "621-DMP3099L-7" (at 165.1 -637.77 0)
+      (effects (font (size 1.27 1.27)) (justify left top) hide)
+    )
+    (property "Mouser Price/Stock" "https://www.mouser.co.uk/ProductDetail/Diodes-Incorporated/DMP3099L-7?qs=L1DZKBg7t5HhdiZT7qYxFw%3D%3D" (at 165.1 -737.77 0)
+      (effects (font (size 1.27 1.27)) (justify left top) hide)
+    )
+    (property "Arrow Part Number" "DMP3099L-7" (at 165.1 -837.77 0)
+      (effects (font (size 1.27 1.27)) (justify left top) hide)
+    )
+    (property "Arrow Price/Stock" "https://www.arrow.com/en/products/dmp3099l-7/diodes-incorporated?region=nac" (at 165.1 -937.77 0)
+      (effects (font (size 1.27 1.27)) (justify left top) hide)
+    )
+    (pin "1")
+    (pin "2")
+    (pin "3")
+    (instances
+      (project "TelescopeController"
+        (path "/3c828e93-3f7d-4aa6-912d-1890319e3f16/979fca36-8703-44d3-91ed-9d630dff4adb"
+          (reference "Q2") (unit 1)
+        )
+        (path "/3c828e93-3f7d-4aa6-912d-1890319e3f16/23dd2fea-7840-477d-ad9b-765c8187b721"
+          (reference "Q10") (unit 1)
+        )
+        (path "/3c828e93-3f7d-4aa6-912d-1890319e3f16/00503a22-69b6-42b3-9f95-98996579316d"
+          (reference "Q11") (unit 1)
+        )
+        (path "/3c828e93-3f7d-4aa6-912d-1890319e3f16/99a9f577-bb8b-4ddf-bf87-90e55a8a0aaf"
+          (reference "Q12") (unit 1)
+        )
+      )
+    )
+  )
   (symbol (lib_id "Connector:TestPoint") (at 161.29 78.74 90) (unit 1)
     (in_bom yes) (on_board yes) (dnp no) (fields_autoplaced)
@@
       (effects (font (size 1.27 1.27)) (justify left))
     )
-    (property "Value" "100R" (at 139.7 52.07 0)
+    (property "Value" "1k" (at 139.7 52.07 0)
       (effects (font (size 1.27 1.27)) (justify left))
     )
@@
   (symbol (lib_id "Device:LED") (at 161.29 99.06 90) (unit 1)
     (in_bom yes) (on_board yes) (dnp no) (fields_autoplaced)
-    (property "Reference" "D3" (at 165.1 99.3775 90)
+    (property "Reference" "D13" (at 165.1 99.3775 90)
       (effects (font (size 1.27 1.27)) (justify right))
     )
-    (property "Value" "SML-LX0805GC-TR" (at 165.1 101.9175 90)
+    (property "Value" "LED" (at 165.1 101.9175 90)
       (effects (font (size 1.27 1.27)) (justify right))
     )
-    (property "Footprint" "LED_SMD:LED_0805_2012Metric_Pad1.15x1.40mm_HandSolder" (at 161.29 99.06 0)
+    (property "Footprint" "LED_THT:LED_D3.0mm" (at 161.29 99.06 0)
       (effects (font (size 1.27 1.27)) hide)
     )
@@
       (project "TelescopeController"
         (path "/3c828e93-3f7d-4aa6-912d-1890319e3f16"
-          (reference "D3") (unit 1)
-        )
-        (path "/3c828e93-3f7d-4aa6-912d-1890319e3f16/979fca36-8703-44d3-91ed-9d630dff4adb"
-          (reference "D4") (unit 1)
-        )
-        (path "/3c828e93-3f7d-4aa6-912d-1890319e3f16/23dd2fea-7840-477d-ad9b-765c8187b721"
-          (reference "D5") (unit 1)
-        )
-        (path "/3c828e93-3f7d-4aa6-912d-1890319e3f16/00503a22-69b6-42b3-9f95-98996579316d"
-          (reference "D6") (unit 1)
-        )
-        (path "/3c828e93-3f7d-4aa6-912d-1890319e3f16/99a9f577-bb8b-4ddf-bf87-90e55a8a0aaf"
-          (reference "D7") (unit 1)
+          (reference "D13") (unit 1)
+        )
+        (path "/3c828e93-3f7d-4aa6-912d-1890319e3f16/979fca36-8703-44d3-91ed-9d630dff4adb"
+          (reference "D12") (unit 1)
+        )
+        (path "/3c828e93-3f7d-4aa6-912d-1890319e3f16/23dd2fea-7840-477d-ad9b-765c8187b721"
+          (reference "D9") (unit 1)
+        )
+        (path "/3c828e93-3f7d-4aa6-912d-1890319e3f16/00503a22-69b6-42b3-9f95-98996579316d"
+          (reference "D8") (unit 1)
+        )
+        (path "/3c828e93-3f7d-4aa6-912d-1890319e3f16/99a9f577-bb8b-4ddf-bf87-90e55a8a0aaf"
+          (reference "D13") (unit 1)
         )
       )
@@
       (effects (font (size 1.27 1.27)) (justify left))
     )
-    (property "Value" "1A" (at 163.83 36.83 0)
+    (property "Value" "1.5A" (at 163.83 36.83 0)
       (effects (font (size 1.27 1.27)) (justify left))
     )
@@
         )
       )
-    )
-  )
-  (symbol (lib_id "AO3423:AO3423") (at 153.67 66.04 0) (unit 1)
-    (in_bom yes) (on_board yes) (dnp no) (fields_autoplaced)
-    (property "Reference" "Q2" (at 165.1 62.23 0)
-      (effects (font (size 1.27 1.27)) (justify left))
-    )
-    (property "Value" "AO3423" (at 165.1 64.77 0)
-      (effects (font (size 1.27 1.27)) (justify left))
-    )
-    (property "Footprint" "AO3423:SOT95P280X125-3N" (at 165.1 164.77 0)
-      (effects (font (size 1.27 1.27)) (justify left top) hide)
-    )
-    (property "Datasheet" "http://www.aosmd.com/pdfs/datasheet/AO3423.pdf" (at 165.1 264.77 0)
-      (effects (font (size 1.27 1.27)) (justify left top) hide)
-    )
-    (property "Height" "1.25" (at 165.1 464.77 0)
-      (effects (font (size 1.27 1.27)) (justify left top) hide)
-    )
-    (property "Manufacturer_Name" "Alpha & Omega Semiconductors" (at 165.1 564.77 0)
-      (effects (font (size 1.27 1.27)) (justify left top) hide)
-    )
-    (property "Manufacturer_Part_Number" "AO3423" (at 165.1 664.77 0)
-      (effects (font (size 1.27 1.27)) (justify left top) hide)
-    )
-    (property "Mouser Part Number" "" (at 165.1 764.77 0)
-      (effects (font (size 1.27 1.27)) (justify left top) hide)
-    )
-    (property "Mouser Price/Stock" "" (at 165.1 864.77 0)
-      (effects (font (size 1.27 1.27)) (justify left top) hide)
-    )
-    (property "Arrow Part Number" "AO3423" (at 165.1 964.77 0)
-      (effects (font (size 1.27 1.27)) (justify left top) hide)
-    )
-    (property "Arrow Price/Stock" "https://www.arrow.com/en/products/ao3423/alpha-and-omega-semiconductor?region=europe" (at 165.1 1064.77 0)
-      (effects (font (size 1.27 1.27)) (justify left top) hide)
-    )
-    (pin "1")
-    (pin "2")
-    (pin "3")
-    (instances
-      (project "TelescopeController"
-        (path "/3c828e93-3f7d-4aa6-912d-1890319e3f16"
-          (reference "Q2") (unit 1)
-        )
-        (path "/3c828e93-3f7d-4aa6-912d-1890319e3f16/979fca36-8703-44d3-91ed-9d630dff4adb"
-          (reference "Q2") (unit 1)
-        )
-        (path "/3c828e93-3f7d-4aa6-912d-1890319e3f16/23dd2fea-7840-477d-ad9b-765c8187b721"
-          (reference "Q4") (unit 1)
-        )
-        (path "/3c828e93-3f7d-4aa6-912d-1890319e3f16/00503a22-69b6-42b3-9f95-98996579316d"
-          (reference "Q6") (unit 1)
-        )
-        (path "/3c828e93-3f7d-4aa6-912d-1890319e3f16/99a9f577-bb8b-4ddf-bf87-90e55a8a0aaf"
-          (reference "Q8") (unit 1)
-        )
-      )
