File: TelescopeController/ControlSW.kicad_sch (KiCad schematic)
At the start: 3 parts

Commit message: add telescope controller v2
Parts:
- removed S2: AS1E-5M-10-Z, AS1E-5M-10-Z:AS1E5M10Z, symbol AS1E-5M-10-Z:AS1E-5M-10-Z
- added S8: AS1E-2M-10-Z, AS1E-2M-10-Z:AS1E2M10Z, symbol AS1E-2M-10-Z:AS1E-2M-10-Z
Connections:
- net +5V: now also S8.2
- net OFF: now also S8.3
- net ON: now also S8.1
Changed lines of the file:
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@@
     )
   )
-  (symbol (lib_id "AS1E-5M-10-Z:AS1E-5M-10-Z") (at 104.14 96.52 0) (unit 1)
+  (symbol (lib_id "AS1E-2M-10-Z:AS1E-2M-10-Z") (at 127 96.52 0) (mirror y) (unit 1)
     (in_bom yes) (on_board yes) (dnp no)
-    (property "Reference" "S2" (at 124.46 176.53 0)
-      (effects (font (size 1.27 1.27)) hide)
-    )
-    (property "Value" "AS1E-5M-10-Z" (at 115.57 91.44 0)
+    (property "Reference" "S8" (at 116.84 109.22 0)
       (effects (font (size 1.27 1.27)))
     )
-    (property "Footprint" "AS1E-5M-10-Z:AS1E5M10Z" (at 123.19 191.44 0)
+    (property "Value" "AS1E-2M-10-Z" (at 116.84 106.68 0)
+      (effects (font (size 1.27 1.27)))
+    )
+    (property "Footprint" "AS1E-2M-10-Z:AS1E2M10Z" (at 110.49 191.44 0)
       (effects (font (size 1.27 1.27)) (justify left top) hide)
     )
-    (property "Datasheet" "https://www.nidec-copal-electronics.com/e/catalog/switch/as.pdf" (at 123.19 291.44 0)
+    (property "Datasheet" "https://www.nidec-copal-electronics.com/e/catalog/switch/as.pdf" (at 110.49 291.44 0)
       (effects (font (size 1.27 1.27)) (justify left top) hide)
     )
-    (property "Height" "5" (at 123.19 491.44 0)
+    (property "Height" "12.3" (at 110.49 491.44 0)
       (effects (font (size 1.27 1.27)) (justify left top) hide)
     )
-    (property "Manufacturer_Name" "NIDEC COPAL" (at 123.19 591.44 0)
+    (property "Manufacturer_Name" "Nidec Copal" (at 110.49 591.44 0)
       (effects (font (size 1.27 1.27)) (justify left top) hide)
     )
-    (property "Manufacturer_Part_Number" "AS1E-5M-10-Z" (at 123.19 691.44 0)
+    (property "Manufacturer_Part_Number" "AS1E-2M-10-Z" (at 110.49 691.44 0)
       (effects (font (size 1.27 1.27)) (justify left top) hide)
     )
-    (property "Mouser Part Number" "" (at 123.19 791.44 0)
+    (property "Mouser Part Number" "229-AS1E-2M-10-Z" (at 110.49 791.44 0)
       (effects (font (size 1.27 1.27)) (justify left top) hide)
     )
-    (property "Mouser Price/Stock" "" (at 123.19 891.44 0)
+    (property "Mouser Price/Stock" "https://www.mouser.co.uk/ProductDetail/Nidec-Copal/AS1E-2M-10-Z?qs=XeJtXLiO41SfK19XCq4wJw%3D%3D" (at 110.49 891.44 0)
       (effects (font (size 1.27 1.27)) (justify left top) hide)
     )
-    (property "Arrow Part Number" "" (at 123.19 991.44 0)
+    (property "Arrow Part Number" "" (at 110.49 991.44 0)
       (effects (font (size 1.27 1.27)) (justify left top) hide)
     )
-    (property "Arrow Price/Stock" "" (at 123.19 1091.44 0)
+    (property "Arrow Price/Stock" "" (at 110.49 1091.44 0)
       (effects (font (size 1.27 1.27)) (justify left top) hide)
     )
@@
     (pin "2")
     (pin "3")
-    (pin "B1")
-    (pin "B2")
     (instances
       (project "TelescopeController"
-        (path "/3c828e93-3f7d-4aa6-912d-1890319e3f16"
-          (reference "S2") (unit 1)
-        )
         (path "/3c828e93-3f7d-4aa6-912d-1890319e3f16/bd7eb281-3960-400d-ae01-b66be830f556"
-          (reference "S5") (unit 1)
+          (reference "S8") (unit 1)
         )
         (path "/3c828e93-3f7d-4aa6-912d-1890319e3f16/6daebbe9-58c7-47f2-8f6b-aa832be29fb8"
-          (reference "S2") (unit 1)
+          (reference "S4") (unit 1)
         )
         (path "/3c828e93-3f7d-4aa6-912d-1890319e3f16/515f19a6-a884-4329-bdf3-4bdeab9c8c9f"
-          (reference "S6") (unit 1)
+          (reference "S7") (unit 1)
         )
         (path "/3c828e93-3f7d-4aa6-912d-1890319e3f16/ebb5a353-9537-42a9-911d-23b896ea5a0a"
-          (reference "S1") (unit 1)
+          (reference "S10") (unit 1)
         )
         (path "/3c828e93-3f7d-4aa6-912d-1890319e3f16/19a93400-7d67-40e8-abcb-d6bbaaf6204c"
-          (reference "S3") (unit 1)
+          (reference "S9") (unit 1)
         )
       )
