File: TelescopeController/TelescopeController.kicad_sch (KiCad schematic)
At the start: 24 parts, among them J1 PJ-102BH, J10 Screw_Terminal_01x02, J2 RCJ-041, J3 RCJ-041, J4 RCJ-041, J5 Conn_01x03_Pin, J6 Screw_Terminal_01x02, J7 Screw_Terminal_01x02, J8 Screw_Terminal_01x02, J9 Screw_Terminal_01x02

Commit message: add telescope controller v2
Parts:
- removed D1, D2, D3: SML-LX0805GC-TR, LED_SMD:LED_0805_2012Metric_Pad1.15x1.40mm_HandSolder, symbol Device:LED
- removed J10, J6, J7, J8, J9: Screw_Terminal_01x02, OSTVN02A150:OSTVN02A150, symbol Connector:Screw_Terminal_01x02
- removed VR1, VR4, VR5: PTD901-1015K-B103, PTD901-1015K-B103:PTD9011015KB103, symbol PTD901-1015K-B103:PTD901-1015K-B103
- added D10, D11, D14: LED, LED_THT:LED_D3.0mm, symbol Device:LED
- added J1: PJ-102BH, PJ-102BH:PJ-102AH, symbol PJ-102BH:PJ-102BH
- added J11: Conn_02x04_Counter_Clockwise, Connector_PinHeader_2.54mm:PinHeader_2x04_P2.54mm_Horizontal, symbol Connector_Generic:Conn_02x04_Counter_Clockwise
- R1: value 490R -> 1k
- R1: value 140R -> 300R
- renumbered J1 to J7
Connections:
- net 12V_SWITCHING3/OUT: now also J1.1
- net GND: now also D10.1 (K), D11.1 (K), D14.1 (K), J1.2, J1.3
- net HEATER1_OFF: now also A1.19 (A0); no longer A1.1 (D1/TX)
- net HEATER1_ON: now also A1.20 (A1); no longer A1.2 (D0/RX)
- net Thermistor/THERM+: now also J11.4 (Pin_4)
- net Thermistor/THERM-: now also J11.3 (Pin_3)
- net Thermistor1/THERM+: now also J11.2 (Pin_2)
- net Thermistor1/THERM-: now also J11.1 (Pin_1)
- net Thermistor2/THERM+: now also J11.8 (Pin_8)
- net Thermistor2/THERM-: now also J11.7 (Pin_7)
- net Thermistor3/THERM+: now also J11.6 (Pin_6)
- net Thermistor3/THERM-: now also J11.5 (Pin_5)
- net at R1.2: now also D10.2 (A)
- net at R1.2: now also D11.2 (A)
- net at R1.2: now also D14.2 (A)
Other:
- note added: "HEATER 1"
- note added: "HEATER 2"
- note added: "HEATER 3"
- note removed: "TODO: confirm nano pinout"
