File: TelescopeController/thermistor.kicad_sch (KiCad schematic)
At the start: 1 part

Commit message: add telescope controller v2
Parts:
- R1: value 10k -> 10k, 0.1%
Changed lines of the file:
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@@
       (effects (font (size 1.27 1.27)) (justify left))
     )
-    (property "Value" "10k" (at 137.16 99.822 0)
+    (property "Value" "10k, 0.1%" (at 137.16 99.822 0)
       (effects (font (size 1.27 1.27)) (justify left))
     )
